File: 06-MiniBLE/06-MiniBLE.kicad_sch (KiCad schematic)
At the start: 23 parts, among them J1 Conn_01x10, U1 ICM-20602, Y1 Crystal

Commit message: Updating layout for wand
Parts:
- added D5: LED_ARGB, LED_SMD:LED_Lumex_SML-LX0303SIUPGUSB, symbol Device:LED_ARGB
- added R5: 1k, Resistor_SMD:R_0402_1005Metric_Pad0.72x0.64mm_HandSolder, symbol Device:R_US
Connections:
- net +BATT: now also R5.1
- net GYRO_CS: now also E1.16 (P0.03); no longer E1.19 (P0.06)
- net LED4B: now also E1.8 (P0.31); no longer E1.4 (P0.27)
- net LED4G: now also E1.7 (P0.30); no longer E1.3 (P0.26)
- net LED4R: now also E1.6 (P0.29); no longer E1.2 (P0.25)
- net SPI_CLK: now also E1.19 (P0.06); no longer E1.18 (P0.05)
- net SPI_MISO: now also E1.17 (P0.04); no longer E1.16 (P0.03)
- net SPI_MOSI: now also E1.18 (P0.05); no longer E1.17 (P0.04)
- net LED5R: now reaches E1.30 (P0.16)
- net LED5R: now also D5.2 (RK)
- net LED5G: now reaches E1.31 (P0.17)
- net LED5G: now also D5.3 (GK)
- net LED5B: now reaches E1.32 (P0.18)
- net LED5B: now also D5.4 (BK)
- new net: D5.1 (A), R5.2
Changed lines of the file:
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@@
 (kicad_sch (version 20201015) (generator eeschema)
-  (page 1 1)
   (paper "A4")
   (junction (at 86.36 115.57) (diameter 0.9144) (color 0 0 0 0))
@@
   (junction (at 224.79 63.5) (diameter 0.9144) (color 0 0 0 0))
   (junction (at 236.22 63.5) (diameter 0.9144) (color 0 0 0 0))
+  (no_connect (at 99.06 134.62))
+  (no_connect (at 205.74 69.85))
+  (no_connect (at 99.06 137.16))
   (no_connect (at 154.94 90.17))
-  (no_connect (at 99.06 134.62))
-  (no_connect (at 99.06 137.16))
-  (no_connect (at 205.74 69.85))
   (wire (pts (xy 46.99 60.96) (xy 59.69 60.96))
     (stroke (width 0) (type solid) (color 0 0 0 0))
@@
     (stroke (width 0) (type solid) (color 0 0 0 0))
   )
+  (wire (pts (xy 205.74 85.09) (xy 217.17 85.09))
+    (stroke (width 0) (type solid) (color 0 0 0 0))
+  )
+  (wire (pts (xy 205.74 87.63) (xy 217.17 87.63))
+    (stroke (width 0) (type solid) (color 0 0 0 0))
+  )
+  (wire (pts (xy 205.74 90.17) (xy 217.17 90.17))
+    (stroke (width 0) (type solid) (color 0 0 0 0))
+  )
   (wire (pts (xy 205.74 95.25) (xy 217.17 95.25))
     (stroke (width 0) (type solid) (color 0 0 0 0))
@@
     (stroke (width 0) (type solid) (color 0 0 0 0))
   )
-  (wire (pts (xy 205.74 107.95) (xy 217.17 107.95))
-    (stroke (width 0) (type solid) (color 0 0 0 0))
-  )
-  (wire (pts (xy 205.74 110.49) (xy 217.17 110.49))
-    (stroke (width 0) (type solid) (color 0 0 0 0))
-  )
-  (wire (pts (xy 205.74 113.03) (xy 217.17 113.03))
+  (wire (pts (xy 205.74 118.11) (xy 217.17 118.11))
+    (stroke (width 0) (type solid) (color 0 0 0 0))
+  )
+  (wire (pts (xy 205.74 120.65) (xy 217.17 120.65))
+    (stroke (width 0) (type solid) (color 0 0 0 0))
+  )
+  (wire (pts (xy 205.74 123.19) (xy 217.17 123.19))
     (stroke (width 0) (type solid) (color 0 0 0 0))
   )
@@
     (stroke (width 0) (type solid) (color 0 0 0 0))
   )
+  (wire (pts (xy 227.33 43.18) (xy 227.33 50.8))
+    (stroke (width 0) (type solid) (color 0 0 0 0))
+  )
+  (wire (pts (xy 232.41 43.18) (xy 232.41 50.8))
+    (stroke (width 0) (type solid) (color 0 0 0 0))
+  )
   (wire (pts (xy 236.22 62.23) (xy 236.22 63.5))
     (stroke (width 0) (type solid) (color 0 0 0 0))
   )
+  (wire (pts (xy 237.49 43.18) (xy 237.49 50.8))
+    (stroke (width 0) (type solid) (color 0 0 0 0))
+  )
   (label "SWDCLK" (at 48.26 63.5 0)
     (effects (font (size 1.27 1.27)) (justify left bottom))
@@
     (effects (font (size 1.27 1.27)) (justify right bottom))
   )
-  (label "SPI_MISO" (at 143.51 92.71 0)
-    (effects (font (size 1.27 1.27)) (justify left bottom))
-  )
-  (label "SPI_MOSI" (at 143.51 95.25 0)
-    (effects (font (size 1.27 1.27)) (justify left bottom))
-  )
-  (label "SPI_CLK" (at 143.51 97.79 0)
-    (effects (font (size 1.27 1.27)) (justify left bottom))
-  )
-  (label "GYRO_CS" (at 143.51 100.33 0)
+  (label "GYRO_CS" (at 143.51 92.71 0)
+    (effects (font (size 1.27 1.27)) (justify left bottom))
+  )
+  (label "SPI_MISO" (at 143.51 95.25 0)
+    (effects (font (size 1.27 1.27)) (justify left bottom))
+  )
+  (label "SPI_MOSI" (at 143.51 97.79 0)
+    (effects (font (size 1.27 1.27)) (justify left bottom))
+  )
+  (label "SPI_CLK" (at 143.51 100.33 0)
     (effects (font (size 1.27 1.27)) (justify left bottom))
   )
@@
     (effects (font (size 1.27 1.27)) (justify right bottom))
   )
-  (label "LED4R" (at 207.01 107.95 0)
-    (effects (font (size 1.27 1.27)) (justify left bottom))
-  )
-  (label "LED4G" (at 207.01 110.49 0)
-    (effects (font (size 1.27 1.27)) (justify left bottom))
-  )
-  (label "LED4B" (at 207.01 113.03 0)
+  (label "LED4R" (at 207.01 118.11 0)
+    (effects (font (size 1.27 1.27)) (justify left bottom))
+  )
+  (label "LED4G" (at 207.01 120.65 0)
+    (effects (font (size 1.27 1.27)) (justify left bottom))
+  )
+  (label "LED4B" (at 207.01 123.19 0)
     (effects (font (size 1.27 1.27)) (justify left bottom))
   )
   (label "NRF_RST" (at 208.28 97.79 0)
     (effects (font (size 1.27 1.27)) (justify left bottom))
+  )
+  (label "LED5R" (at 213.36 85.09 180)
+    (effects (font (size 1.27 1.27)) (justify right bottom))
+  )
+  (label "LED5G" (at 213.36 87.63 180)
+    (effects (font (size 1.27 1.27)) (justify right bottom))
+  )
+  (label "LED5B" (at 213.36 90.17 180)
+    (effects (font (size 1.27 1.27)) (justify right bottom))
+  )
+  (label "LED5R" (at 227.33 44.45 270)
+    (effects (font (size 1.27 1.27)) (justify right bottom))
+  )
+  (label "LED5G" (at 232.41 44.45 270)
+    (effects (font (size 1.27 1.27)) (justify right bottom))
+  )
+  (label "LED5B" (at 237.49 44.45 270)
+    (effects (font (size 1.27 1.27)) (justify right bottom))
   )
   (symbol (lib_id "power:+BATT") (at 59.69 60.96 0) (unit 1)
@@
     )
   )
+  (symbol (lib_id "power:+BATT") (at 232.41 25.4 0) (unit 1)
+    (in_bom yes) (on_board yes)
+    (property "Reference" "#PWR01" (id 0) (at 232.41 29.21 0)
+      (effects (font (size 1.27 1.27)) hide)
+    )
+    (property "Value" "+BATT" (id 1) (at 233.68 21.59 0))
+    (property "Footprint" "" (id 2) (at 232.41 25.4 0)
+      (effects (font (size 1.27 1.27)) hide)
+    )
+    (property "Datasheet" "" (id 3) (at 232.41 25.4 0)
+      (effects (font (size 1.27 1.27)) hide)
+    )
+  )
   (symbol (lib_id "power:+BATT") (at 236.22 62.23 0) (unit 1)
     (in_bom yes) (on_board yes)
@@
     )
   )
+  (symbol (lib_id "Device:R_US") (at 232.41 29.21 0) (unit 1)
+    (in_bom yes) (on_board yes)
+    (property "Reference" "R5" (id 0) (at 234.95 27.94 0)
+      (effects (font (size 1.27 1.27)) (justify left))
+    )
+    (property "Value" "1k" (id 1) (at 234.95 29.21 0)
+      (effects (font (size 1.27 1.27)) (justify left))
+    )
+    (property "Footprint" "Resistor_SMD:R_0402_1005Metric_Pad0.72x0.64mm_HandSolder" (id 2) (at 233.426 29.464 90)
+      (effects (font (size 1.27 1.27)) hide)
+    )
+    (property "Datasheet" "~" (id 3) (at 232.41 29.21 0)
+      (effects (font (size 1.27 1.27)) hide)
+    )
+  )
   (symbol (lib_id "Device:C_Small") (at 86.36 92.71 0) (unit 1)
     (in_bom yes) (on_board yes)
@@
     )
     (property "Datasheet" "~" (id 3) (at 203.2 38.1 0)
+      (effects (font (size 1.27 1.27)) hide)
+    )
+  )
+  (symbol (lib_id "Device:LED_ARGB") (at 232.41 38.1 90) (unit 1)
+    (in_bom yes) (on_board yes)
+    (property "Reference" "D5" (id 0) (at 241.3 36.83 90)
+      (effects (font (size 1.27 1.27)) (justify right))
+    )
+    (property "Value" "LED_ARGB" (id 1) (at 241.3 38.1 90)
+      (effects (font (size 1.27 1.27)) (justify right))
+    )
+    (property "Footprint" "LED_SMD:LED_Lumex_SML-LX0303SIUPGUSB" (id 2) (at 233.68 38.1 0)
+      (effects (font (size 1.27 1.27)) hide)
+    )
+    (property "Datasheet" "~" (id 3) (at 233.68 38.1 0)
       (effects (font (size 1.27 1.27)) hide)
     )
@@
   )
   (symbol_instances
+    (path "/d3630e4e-a9e9-40b3-bed5-a5e2149116ac"
+      (reference "#PWR01") (unit 1) (value "+BATT") (footprint "")
+    )
     (path "/bb44c0fd-2c59-40a5-bbd9-d01359ceee62"
       (reference "#PWR0101") (unit 1) (value "GND") (footprint "")
@@
       (reference "D4") (unit 1) (value "LED_ARGB") (footprint "LED_SMD:LED_Lumex_SML-LX0303SIUPGUSB")
     )
+    (path "/712f2690-b193-462f-862b-f14095ed84dd"
+      (reference "D5") (unit 1) (value "LED_ARGB") (footprint "LED_SMD:LED_Lumex_SML-LX0303SIUPGUSB")
+    )
     (path "/22f91e4a-db38-4bbe-a1e5-361f0632600f"
       (reference "E1") (unit 1) (value "MDBT42Q-512KV2") (footprint "06-MiniBLE:RAYTAC_MDBT42Q-512KV2")
@@
       (reference "R4") (unit 1) (value "1k") (footprint "Resistor_SMD:R_0402_1005Metric_Pad0.72x0.64mm_HandSolder")
     )
+    (path "/76f75a0c-e5de-4968-893b-02878cf4dd7b"
+      (reference "R5") (unit 1) (value "1k") (footprint "Resistor_SMD:R_0402_1005Metric_Pad0.72x0.64mm_HandSolder")
+    )
     (path "/0cc9c233-b26c-47da-8d63-48672ead1a14"

Commit message: Day 7 - layout for miniBLE wand
Parts:
- removed J1: Conn_01x10, Connector_PinHeader_2.54mm:PinHeader_1x10_P2.54mm_Vertical, symbol Connector_Generic:Conn_01x10
- added J1: TagConnect, Connector:Tag-Connect_TC2030-IDC-NL_2x03_P1.27mm_Vertical, symbol Connector:Conn_01x06_Male
- added TP1, TP2, TP3, TP4: TestPoint, TestPoint:TestPoint_Pad_1.0x1.0mm, symbol Connector:TestPoint
Connections:
- net +BATT: now also J1.1 (Pin_1)
- net GND: now also J1.5 (Pin_5)
- net GYRO_CS: now also TP4.1
- net LED1B: now also E1.20 (P0.07); no longer E1.22 (P0.09)
- net LED1G: now also E1.22 (P0.09); no longer E1.21 (P0.08)
- net LED1R: now also E1.21 (P0.08); no longer E1.20 (P0.07)
- net LED2B: now also E1.23 (P0.10); no longer E1.26 (P0.12)
- net LED2G: now also E1.26 (P0.12); no longer E1.25 (P0.11)
- net LED2R: now also E1.25 (P0.11); no longer E1.23 (P0.10)
- net LED3B: now also E1.27 (P0.13); no longer E1.29 (P0.15)
- net LED3G: now also E1.29 (P0.15); no longer E1.28 (P0.14)
- net LED3R: now also E1.28 (P0.14); no longer E1.27 (P0.13)
- net LED4B: now also D5.4 (BK); no longer D4.4 (BK)
- net LED4G: now also D5.3 (GK); no longer D4.3 (GK)
- net LED4R: now also D5.2 (RK); no longer D4.2 (RK)
- net LED5B: now also D4.4 (BK), E1.30 (P0.16); no longer D5.4 (BK), E1.32 (P0.18)
- net LED5G: now also D4.3 (GK); no longer D5.3 (GK)
- net LED5R: now also D4.2 (RK), E1.32 (P0.18); no longer D5.2 (RK), E1.30 (P0.16)
- net NRF_RST: now also J1.4 (Pin_4)
- net SPI_CLK: now also TP3.1
- net SPI_MISO: now also TP1.1
- net SPI_MOSI: now also TP2.1
- net SWDCLK: now also J1.3 (Pin_3)
- net SWDIO: now also J1.2 (Pin_2)
- no-connect marks 4 -> 5
